File: BOARD/Frontend_test/_autosave-Frontend_test.sch (KiCad schematic (older format))
At the start: 47 parts, among them J1 Conn_Coaxial, J2 Conn_01x02, J3 Conn_02x10_Top_Bottom, J4 Conn_01x03, SW1 SW_Push, U1 AD8253, U2 MCP33131D, U3 AP2114-1.8, U4 LT3032-15, U5 AD8675, U6 REF5050AD

Commit message: More work on final Schematic. Power, digital and output section close to final. No frontend yet.
Parts:
- removed SW1: SW_Push, symbol Switch:SW_Push
Changed lines of the file:
@@
 	10950 5300 10850 5300
 Connection ~ 10850 5500
-$Comp
-L Switch:SW_Push SW1
-U 1 1 5D883389
-P 7500 1300
-F 0 "SW1" H 7500 1585 50  0000 C CNN
-F 1 "SW_Push" H 7500 1494 50  0000 C CNN
-F 2 "" H 7500 1500 50  0001 C CNN
-F 3 "~" H 7500 1500 50  0001 C CNN
-	1    7500 1300
-	1    0    0    -1
-$EndComp
 $EndSCHEMATC
