File: BOARD/SingularitySurfer_V1/Frontend.sch (KiCad schematic (older format))
At the start: 0 parts

Commit message: Final Board schematic almost done and started on layout
Parts:
- added C33, C34: 10u, Capacitor_SMD:C_0805_2012Metric_Pad1.15x1.40mm_HandSolder, symbol Device:C
- added C35: 1u, Capacitor_SMD:C_1206_3216Metric_Pad1.42x1.75mm_HandSolder, symbol Device:C
- added C36, C37, C38, C39, C40, C41, C42: C, Capacitor_SMD:C_1206_3216Metric_Pad1.42x1.75mm_HandSolder, symbol Device:C
- added D13: D_Zener, Diode_SMD:D_SOD-323, symbol Device:D_Zener
- added D14, D15: D_Schottky_x2_Serial_AKC, Package_TO_SOT_SMD:SOT-23, symbol Device:D_Schottky_x2_Serial_AKC
- added J10, J9: Conn_01x02, Connector_PinHeader_2.54mm:PinHeader_1x02_P2.54mm_Vertical, symbol Connector_Generic:Conn_01x02
- added J11, J12: Conn_Coaxial, Connector_Coaxial:SMA_Molex_73251-2200_Horizontal, symbol Connector:Conn_Coaxial
- added R27, R28, R29, R30, R31, R32, R33, R34: R, Resistor_SMD:R_0805_2012Metric_Pad1.15x1.40mm_HandSolder, symbol Device:R
- added U10: REF5050AD, Package_SO:SOIC-8_3.9x4.9mm_P1.27mm, symbol Reference_Voltage:REF5050AD
- added U11: AD8675, Package_SO:MSOP-8_3x3mm_P0.65mm, symbol SingularitySurfer:AD8675
- added U12: AD8253, Package_SO:MSOP-10_3x3mm_P0.5mm, symbol SingularitySurfer:AD8253
- added U9: MCP33131D, Package_SO:MSOP-10_3x3mm_P0.5mm, symbol SingularitySurfer:MCP33131D
Connections:
- new net: C40.1, R34.1, U12.1 (In_low)
- new net: C39.2, R33.1, U12.10 (In_pos)
- new net: D15.3 (common), R29.1, R32.1, U12.7 (OUT)
- new net: C38.1, D14.3 (common), R30.1, R31.1, U11.6, U12.9 (REF)
- new net: C33.1, C34.1, D13.1 (K), D14.2 (K), D15.2 (K), R28.2, U10.6 (Vout), U9.1 (REF)
- new net: C36.2, J12.1 (In), R29.2, U9.3 (IN_pos)
- new net: C37.2, R30.2, U9.4 (IN_neg)
- new net: C38.2, R31.2, R32.2, U11.2 (-)
- new net: R27.2, R28.1, U11.3 (+)
- new net: C35.2, U10.5 (Trim/NR)
- new net: C41.1, J11.1 (In), J9.1 (Pin_1)
- new net: C42.1, J10.2 (Pin_2), J11.2 (Ext), J9.2 (Pin_2)
- new net: C41.2, R33.2
- new net: C42.2, R34.2
- new net +15V: U10.2 (Vin), U11.7 (V+)
- new net +8V: U12.8 (V_pos)
- new net -15V: U11.4 (V-)
- new net -8V: U12.3 (V_neg), U12.6 (WEn)
- new net 1V8: U9.2 (AVdd)
- new net 3V3: U9.10 (DVIO)
- new net A0: U12.4 (A0)
- new net A1: U12.5 (A1)
- new net CONVST: U9.6 (CONVST)
- new net GNDA: C33.2, C34.2, C35.1, C36.1, C37.1, C39.1, C40.2, D13.2 (A), D14.1 (A), D15.1 (A), J10.1 (Pin_1), J12.2 (Ext), R27.1, U10.4 (GND), U11.1 (NULL), U11.5 (NULL), U12.2 (DGND), U9.5 (GND)
- new net SCLK: U9.8 (SCLK)
- new net SDI: U9.9 (SDI)
- new net SDO: U9.7 (SDO)
- no-connect marks 0 -> 1

Commit message: SignularitiSurfer final boar almost donegit status! Fuuuak this is getting rediculous...
Connections:
- net +15V is gone; now on net +8V: U10.2 (Vin), U11.7 (V+)
- net -15V is gone; now on net -8V: U11.4 (V-)
Changed lines of the file:
@@
 NoConn ~ 3500 3600
 Text GLabel 3200 3300 1    50   Input ~ 0
-+15V
++8V
 Wire Wire Line
 	2600 3700 2700 3700
@@
 $EndComp
 Text GLabel 5900 2900 1    50   Input ~ 0
-+15V
++8V
 Text GLabel 5900 3500 3    50   Input ~ 0
--15V
+-8V
 Wire Wire Line
 	5800 3500 5700 3500

Commit message: idiot me forgot to push final changes half a year ago.. Fixed code: filter constant 3 bit, filter downsampling factor and some mics.   Converted KiCad stuff to new version
Parts:
- U11: symbol SingularitySurfer:AD8675 -> SingularitySurfer_V1-rescue:AD8675-SingularitySurfer
- U12: symbol SingularitySurfer:AD8253 -> SingularitySurfer_V1-rescue:AD8253-SingularitySurfer
- U9: symbol SingularitySurfer:MCP33131D -> SingularitySurfer_V1-rescue:MCP33131D-SingularitySurfer
Changed lines of the file:
@@
 EESchema Schematic File Version 4
-LIBS:SingularitySurfer_V1-cache
 EELAYER 30 0
 EELAYER END
@@
 $EndComp
 $Comp
-L SingularitySurfer:AD8675 U11
+L SingularitySurfer_V1-rescue:AD8675-SingularitySurfer U11
 U 1 1 5D762A93
 P 5800 3200
@@
 $EndComp
 $Comp
-L SingularitySurfer:AD8253 U12
+L SingularitySurfer_V1-rescue:AD8253-SingularitySurfer U12
 U 1 1 5D6EDD01
 P 7500 4800
@@
 $EndComp
 $Comp
-L SingularitySurfer:MCP33131D U9
+L SingularitySurfer_V1-rescue:MCP33131D-SingularitySurfer U9
 U 1 1 5D6EE5E5
 P 1900 4700
